Commit message: work

File: stompy_sim/agents/stompy/description/robot.urdf (robot description, URDF)
Before this commit: robot robot, 151 links, 150 joints
Links:
- link link_left_arm_2_hand_1_camera_mount_1: mass 0.0032944294 -> None
- link link_legs_1_left_leg_1_calf_pulley_1: mass 0.0056355118 -> None
- link link_legs_1_right_leg_1_calf_pulley_1: mass 0.0056355118 -> None
- link link_right_arm_1_hand_1_camera_mount_1: mass 0.0032944294 -> None
